Commit message: create gazebo.launch file for launch robot in gazebo

File: Day6/auc_ws/src/auc_robot/urdf/my_robot.xacro (robot description, xacro)
@@ -175,5 +175,5 @@
       <origin xyz="0 0 0" rpy="0 0 0"/>
       <geometry>
-        <mesh filename="package://my_robot/meshes/hokuyo.dae"/>
+        <mesh filename="package://auc_robot/meshes/hokuyo.dae"/>
       </geometry>
     </visual>
